File: Programator/Programator.kicad_pcb (KiCad board)
At the start: 2 copper layers, 69 parts, among them J1 USB_A, X1 +12 V, X10 p.8-Com, X11 +12 V, X12 GND, X13 +5V, X14 GND, X15 CONN_6, X16 +12 V, X17 GND, X18 +5V, X19 GND, X2 GND, X20 +5V, X21 CONN_6, X22 CONN_9, X3 GND, X4 +5V, X5 p.5-Com, X6 p.2-Com, X7 p.3-Com, X8 p.4-Com, X9 p.7-Com

Commit message: Ввел трассировку
Parts:
- removed X10: p.8-Com, Connector_PinHeader_2.54mm:PinHeader_1x01_P2.54mm_Vertical
- removed X11, X16: +12 V, Connector_PinHeader_2.54mm:PinHeader_1x01_P2.54mm_Vertical
- removed X12, X14, X17, X19: GND, Connector_PinHeader_2.54mm:PinHeader_1x01_P2.54mm_Vertical
- removed X13, X18, X20: +5V, Connector_PinHeader_2.54mm:PinHeader_1x01_P2.54mm_Vertical
- removed X15, X21: CONN_6, Connector_PinHeader_2.54mm:PinHeader_1x01_P2.54mm_Vertical
- removed X22: CONN_9, Connector_PinHeader_2.54mm:PinHeader_2x05_P2.54mm_Vertical
- removed X7: p.3-Com, Connector_PinHeader_2.54mm:PinHeader_1x01_P2.54mm_Vertical
- removed X8: p.4-Com, Connector_PinHeader_2.54mm:PinHeader_1x01_P2.54mm_Vertical
- X1: value +12 V -> CONN_2; footprint Connector_PinHeader_2.54mm:PinHeader_1x01_P2.54mm_Vertical -> Connector_PinHeader_2.54mm:PinHeader_2x03_P2.54mm_Vertical
- X2: value GND -> CONN_2; footprint Connector_PinHeader_2.54mm:PinHeader_1x01_P2.54mm_Vertical -> Connector_PinHeader_2.54mm:PinHeader_1x02_P2.54mm_Vertical
- X3: value GND -> CONN_2; footprint Connector_PinHeader_2.54mm:PinHeader_1x01_P2.54mm_Vertical -> Connector_PinHeader_2.54mm:PinHeader_2x03_P2.54mm_Vertical
- X4: value +5V -> CONN_2; footprint Connector_PinHeader_2.54mm:PinHeader_1x01_P2.54mm_Vertical -> Connector_PinHeader_2.54mm:PinHeader_1x02_P2.54mm_Vertical
- X5: value p.5-Com -> CONN_9; footprint Connector_PinHeader_2.54mm:PinHeader_1x01_P2.54mm_Vertical -> Connector_Dsub:DSUB-9_Male_Horizontal_P2.77x2.84mm_EdgePinOffset4.94mm_Housed_MountingHolesOffset7.48mm
- X6: value p.2-Com -> CONN_6; footprint Connector_PinHeader_2.54mm:PinHeader_1x01_P2.54mm_Vertical -> Connector_IDC:IDC-Header_2x03_P2.54mm_Vertical
- X9: value p.7-Com -> CONN_6; footprint Connector_PinHeader_2.54mm:PinHeader_1x01_P2.54mm_Vertical -> Connector_IDC:IDC-Header_2x03_P2.54mm_Vertical
- moved X9 139.3 mm to (250.0, 46.0)
- moved X3 138.0 mm to (109.5, 165.5), turned to 0 degrees
- moved R13 138.0 mm to (211.0, 66.5)
- moved X4 127.1 mm to (109.5, 146.0)
- moved X6 84.5 mm to (147.0, 149.5)
- moved J1 81.7 mm to (184.0, 55.3), turned to 180 degrees
- moved R9 61.0 mm to (142.0, 171.0)
- moved C8 55.3 mm to (203.2, 48.8), turned to 270 degrees
- moved X5 52.0 mm to (128.5, 91.0), turned to 90 degrees
- moved R16 49.8 mm to (241.0, 62.0)
- moved C5 46.5 mm to (121.5, 150.5)
- moved ZQ3 46.4 mm to (209.8, 48.5)
- moved VD7 44.3 mm to (152.5, 165.5), turned to 180 degrees
- moved X1 40.1 mm to (57.0, 95.5), turned to 0 degrees
- moved R4 38.7 mm to (127.5, 143.5), turned to 180 degrees
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Connections:
- C1 pad 1: GND -> 0V
- C10 pad 1: GND -> 0V1
- C2 pad 1: GND -> 0V
- C3 pad 1: GND -> 0V
- C7 pad 2: +5V -> +5VL
- C8 pad 1: GND -> 0V1
- C8 pad 2: /OSC1 -> /OSC3
- C9 pad 1: GND -> 0V1
- C9 pad 2: /OSC2 -> /OSC4
- DA1 pad 10: GND -> 0V
- DA2 pad 11: Net-(DA2-Pad11) -> /LED4
- DA2 pad 20: +5V -> +5VL
- DA2 pad 3: /LED3 -> Net-(DA2-Pad3)
- DA2 pad 7: /LED4 -> Net-(DA2-Pad7)
- DA2 pad 9: Net-(DA2-Pad9) -> /LED3
- DA3 pad 10: GND -> 0V1
- DA3 pad 12: /LED1 -> /LED5
- DA3 pad 16: /RST -> /RST1
- DA3 pad 17: /MOSI -> /MOSI1
- DA3 pad 18: /MISO -> /MISO1
- DA3 pad 19: /SCK -> /SCK1
- DA3 pad 4: /OSC2 -> /OSC4
- DA3 pad 5: /OSC1 -> /OSC3
- DA3 pad 9: /LED2 -> /LED6
- J1 pad 4: GND -> 0V1
- J1 pad 5: Net-(J1-Pad5) -> 0V1
- R1 pad 1: GND -> 0V
- R11 pad 2: +5V -> +5VL
- R12 pad 2: +5V -> +5VL
- R16 pad 1: /LED1 -> /LED5
- R17 pad 1: /LED2 -> /LED6
- R18 pad 1: /SCK -> /SCK1
- R19 pad 1: /MOSI -> /MOSI1
- R2 pad 1: GND -> 0V
- R3 pad 1: GND -> 0V
- R4 pad 1: +5V -> +5VL
- VD10 pad 1: GND -> 0V1
- VD11 pad 1: GND -> 0V1
- VD8 pad 2: GND -> 0V1
- VD9 pad 2: GND -> 0V1
- X1 pad 1: +12V -> Net-(X1-Pad1)
- X2 pad 1: GND -> +5V
- X3 pad 1: GND -> Net-(X3-Pad1)
- X4 pad 1: +5V -> +5VL
- X5 pad 1: GND -> Net-(X5-Pad1)
- X6 pad 1: Net-(DA1-Pad17) -> +5VL
- X9 pad 1: Net-(VD3-Pad2) -> +5V1
- ZQ3 pad 1: /OSC1 -> /OSC3
- ZQ3 pad 2: /OSC2 -> /OSC4
Routing:
- net 0V1: track 0.00 -> 167.0 mm
- net 0V: track 0.00 -> 150.5 mm, vias 0 -> 2
- net +5V1: track 0.00 -> 95.2 mm, vias 0 -> 1
- net +5VL: track 0.00 -> 93.2 mm
- net GND: track 99.3 -> 135.3 mm, vias 2 -> 1
- net Net-(J1-Pad2): track 0.00 -> 31.3 mm
- net /OSC3: track 0.00 -> 30.5 mm
- net +5V: track 3.87 -> 33.0 mm
- net Net-(J1-Pad3): track 0.00 -> 24.7 mm
- net /MOSI: track 0.00 -> 24.4 mm
- net Net-(R19-Pad2): track 0.00 -> 24.3 mm, vias 0 -> 1
- net /LED6: track 0.00 -> 19.5 mm
- net /RST1: track 0.00 -> 19.4 mm
- net Net-(VD3-Pad2): track 12.8 -> 31.7 mm, vias 0 -> 1
- net /SCK: track 0.00 -> 18.4 mm
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Other:
- net class Default: clearance 0.2 -> 0.5; trace_width 0.25 -> 0.5
- rule trace_clearance: 0.2 -> 0.5
