File: Programator/Programator.sch (KiCad schematic (older format))
At the start: 69 parts, among them J1 USB_A, X1 +12 V, X10 p.8-Com, X11 +12 V, X12 GND, X13 +5V, X14 GND, X15 CONN_6, X16 +12 V, X17 GND, X18 +5V, X19 GND, X2 GND, X20 +5V, X21 CONN_6, X22 CONN_9, X3 GND, X4 +5V, X5 p.5-Com, X6 p.2-Com, X7 p.3-Com, X8 p.4-Com, X9 p.7-Com

Commit message: Ввел трассировку
Parts:
- removed X1, X11, X16: +12 V, Connector_PinHeader_2.54mm:PinHeader_1x01_P2.54mm_Vertical, symbol Connector_Generic_GOST:CON
- removed X10: p.8-Com, Connector_PinHeader_2.54mm:PinHeader_1x01_P2.54mm_Vertical, symbol Connector_Generic_GOST:CON
- removed X12, X14, X17, X19, X2, X3: GND, Connector_PinHeader_2.54mm:PinHeader_1x01_P2.54mm_Vertical, symbol Connector_Generic_GOST:CON
- removed X13, X18, X20, X4: +5V, Connector_PinHeader_2.54mm:PinHeader_1x01_P2.54mm_Vertical, symbol Connector_Generic_GOST:CON
- removed X22: CONN_9, Connector_PinHeader_2.54mm:PinHeader_2x05_P2.54mm_Vertical, symbol Connector_Generic_GOST:CONN_9
- removed X5: p.5-Com, Connector_PinHeader_2.54mm:PinHeader_1x01_P2.54mm_Vertical, symbol Connector_Generic_GOST:CON
- removed X6: p.2-Com, Connector_PinHeader_2.54mm:PinHeader_1x01_P2.54mm_Vertical, symbol Connector_Generic_GOST:CON
- removed X7: p.3-Com, Connector_PinHeader_2.54mm:PinHeader_1x01_P2.54mm_Vertical, symbol Connector_Generic_GOST:CON
- removed X8: p.4-Com, Connector_PinHeader_2.54mm:PinHeader_1x01_P2.54mm_Vertical, symbol Connector_Generic_GOST:CON
- removed X9: p.7-Com, Connector_PinHeader_2.54mm:PinHeader_1x01_P2.54mm_Vertical, symbol Connector_Generic_GOST:CON
- added X1, X3: CONN_2, Connector_PinHeader_2.54mm:PinHeader_2x03_P2.54mm_Vertical, symbol Connector_Generic_GOST:CONN_6
- added X2, X4: CONN_2, Connector_PinHeader_2.54mm:PinHeader_1x02_P2.54mm_Vertical, symbol Connector_Generic_GOST:CONN_2
- added X5: CONN_9, Connector_Dsub:DSUB-9_Male_Horizontal_P2.77x2.84mm_EdgePinOffset4.94mm_Housed_MountingHolesOffset7.48mm, symbol Connector_Generic_GOST:CONN_9
- X6: renamed from X15; footprint Connector_PinHeader_2.54mm:PinHeader_1x01_P2.54mm_Vertical -> Connector_IDC:IDC-Header_2x03_P2.54mm_Vertical
- X9: renamed from X21; footprint Connector_PinHeader_2.54mm:PinHeader_1x01_P2.54mm_Vertical -> Connector_IDC:IDC-Header_2x03_P2.54mm_Vertical
Connections:
- net +5V: now also X2.1; no longer C7.2, DA2.20 (VCC), R11.2, R12.2, R4.1, X6.1
- net GND: now also X3.2, X3.4, X3.6, X4.2; no longer C1.1, C10.1, C2.1, C3.1, C8.1, C9.1, DA1.10 (GND), DA3.10 (GND), J1.4 (GND), R1.1, R2.1, R3.1, VD10.1 (K), VD11.1 (K), VD8.2 (A), VD9.2 (A), X9.6
- net LED1: no longer DA3.12 (PB0), R16.1
- net LED2: no longer DA3.9 (PD5), R17.1
- net LED3: now also DA2.9 (PD5); no longer DA2.3 (PD1)
- net LED4: now also DA2.11 (PD6); no longer DA2.7 (PD3)
- net MISO: no longer DA3.18 (PB6), X9.3
- net MOSI: no longer DA3.17 (PB5), R19.1
- net OSC1: no longer C8.2, DA3.5 (PA0/XTAL1), ZQ3.1
- net OSC2: no longer C9.2, DA3.4 (PA1/XTAL2), ZQ3.2
- net RST: no longer DA3.16 (PB4), X9.5
- net SCK: no longer DA3.19 (PB7), R18.1
- net at DA1.17 (PB5), R1.2, R5.1: now also X5.2
- net at R8.2: now also X5.8
- net at VD1.2 (A): now also X5.3
- net at VD2.2 (A): now also X5.4
- net at VD3.2 (A): now also X5.7
- net 0V1: now reaches J1.5 (Shield)
- net 0V1: now also C10.1, C8.1, C9.1, DA3.10 (GND), J1.4 (GND), VD10.1 (K), VD11.1 (K), VD8.2 (A), VD9.2 (A), X9.6
- new net: X1.1, X1.3, X1.5
- new net: X3.1, X3.3, X3.5
- new net +5VL: C7.2, DA2.20 (VCC), R11.2, R12.2, R4.1, X4.1, X6.1
- new net 0V: C1.1, C2.1, C3.1, DA1.10 (GND), R1.1, R2.1, R3.1, X1.2, X1.4, X1.6, X2.2, X5.5
- new net LED5: DA3.12 (PB0), R16.1
- new net LED6: DA3.9 (PD5), R17.1
- new net MISO1: DA3.18 (PB6), X9.3
- new net MOSI1: DA3.17 (PB5), R19.1
- new net OSC3: C8.2, DA3.5 (PA0/XTAL1), ZQ3.1
- new net OSC4: C9.2, DA3.4 (PA1/XTAL2), ZQ3.2
- new net RST1: DA3.16 (PB4), X9.5
- new net SCK1: DA3.19 (PB7), R18.1
Other:
- moved on the sheet: C1, C2, C3, DA1, R1, R2, R3, R5, R6, R7, R8, VD1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
