File: EP-528_ser.2/EP-528_ser.2/EP-528_ser.2.sch (KiCad schematic (older format))
At the start: 46 parts, among them X1 CON, X10 CON, X14 CON, X15 CON, X16 CON, X22 CON, X23 CON, X32 CON, X44 CON, X46 CON, X47 CON, X5 CON, X9 CON

Commit message: Обновлены файлы ЭП
Parts:
- removed D1, D2, D4: 140УД20, Package_CDFP_RU:401.14-5, symbol Amplifier_Operational_GOST:140УД20
- added DA1, DA2: 140УД6А, Package_TO_SOT_THT_RU:3101.8, symbol Amplifier_Operational_GOST:140УД6А
- added DA4: 544УД1А, Package_TO_SOT_THT_RU:3101.8, symbol Amplifier_Operational_GOST:140УД6А
- C2: value C -> 47
- C3: value C -> 15
- C8: value C -> 1
- C9: value C -> 6.8
- R11: value R -> 24k
- R12: value R -> 56.2k
- R13: value R -> 33.2k
- R14, R7: value R -> 10k
- R15: value R -> 2.05k
- R2: value R -> 1k
- R20, R22: value R -> 5.05k
- R25: value R -> 82.5k
- R28: value R -> 8.2M
- R29: value R -> 10M
- R36: value R -> 1.01k
- R37: value R -> 2k
- R43: value R -> 2.91k
- R50: value R -> 3.92k
- R54, R55: value R -> 130
- R6: value R -> 180k
- R8: value R -> 12k
- R9: value R -> 8.06k
- R98: value R -> 2M
- VD1, VD10, VD4, VD9: value VD -> 2Д522Б
Changed lines of the file:
@@
 EESchema Schematic File Version 4
-LIBS:EP-528_ser.2-cache
 EELAYER 30 0
 EELAYER END
@@
 P 10550 1600
 F 0 "C8" V 10450 1700 79  0000 L CNN
-F 1 "C" V 10650 1700 79  0000 L CNN
+F 1 "1" V 10650 1700 79  0000 L CNN
 F 2 "" H 10475 1600 60  0001 C CNN
 F 3 "" H 10575 1700 60  0001 C CNN
@@
 P 11300 1600
 F 0 "R37" H 11400 1800 79  0000 C CNN
-F 1 "R" H 11300 1600 79  0000 C CNN
+F 1 "2k" H 11300 1600 79  0000 C CNN
 F 2 "" H 11200 1625 60  0001 C CNN
 F 3 "" H 11325 1425 60  0001 C CNN
@@
 P 2200 2200
 F 0 "R2" H 2200 2350 79  0000 C CNN
-F 1 "R" H 2200 2200 79  0000 C CNN
+F 1 "1k" H 2200 2200 79  0000 C CNN
 F 2 "" H 2100 2225 60  0001 C CNN
 F 3 "" H 2225 2025 60  0001 C CNN
@@
 P 3200 2200
 F 0 "R9" H 3200 2350 79  0000 C CNN
-F 1 "R" H 3200 2200 79  0000 C CNN
+F 1 "8.06k" H 3200 2200 79  0000 C CNN
 F 2 "" H 3100 2225 60  0001 C CNN
 F 3 "" H 3225 2025 60  0001 C CNN
@@
 P 2700 2750
 F 0 "C2" H 2750 2850 79  0000 L CNN
-F 1 "C" H 2800 2650 79  0000 L CNN
+F 1 "47" H 2800 2650 79  0000 L CNN
 F 2 "" H 2625 2750 60  0001 C CNN
 F 3 "" H 2725 2850 60  0001 C CNN
@@
 P 3200 3200
 F 0 "R7" H 3200 3350 79  0000 C CNN
-F 1 "R" H 3200 3200 79  0000 C CNN
+F 1 "10k" H 3200 3200 79  0000 C CNN
 F 2 "" H 3100 3225 60  0001 C CNN
 F 3 "" H 3225 3025 60  0001 C CNN
@@
 P 3900 2650
 F 0 "VD1" V 3900 2796 79  0000 L CNN
-F 1 "VD" H 3900 2450 79  0001 C CNN
+F 1 "2Д522Б" H 3900 2450 79  0001 C CNN
 F 2 "" H 3802 2650 79  0001 C CNN
 F 3 "" H 3802 2650 79  0001 C CNN
@@
 P 4450 2650
 F 0 "VD4" V 4450 2504 79  0000 R CNN
-F 1 "VD" H 4450 2450 79  0001 C CNN
+F 1 "2Д522Б" H 4450 2450 79  0001 C CNN
 F 2 "" H 4352 2650 79  0001 C CNN
 F 3 "" H 4352 2650 79  0001 C CNN
@@
 $EndComp
 $Comp
-L Amplifier_Operational_GOST:140УД20 D1
-U 1 1 67D10D65
-P 5500 2800
-F 0 "D1" H 5500 3495 79  0000 C CNN
-F 1 "140УД20" H 5500 2100 79  0001 C CNN
-F 2 "Package_CDFP_RU:401.14-5" H 5550 1950 79  0001 C CNN
-F 3 "http://www.voshod-krlz.ru/files/datasheets/140UD20.pdf" H 6500 2850 79  0001 C CNN
-	1    5500 2800
-	1    0    0    -1
-$EndComp
-$Comp
 L Device_GOST:R R25
 U 1 1 67D13EBB
 P 5700 1750
 F 0 "R25" H 5700 1900 79  0000 C CNN
-F 1 "R" H 5700 1750 79  0000 C CNN
+F 1 "82.5k" H 5700 1750 79  0000 C CNN
 F 2 "" H 5600 1775 60  0001 C CNN
 F 3 "" H 5725 1575 60  0001 C CNN
@@
 P 2950 4400
 F 0 "R11" H 2950 4550 79  0000 C CNN
-F 1 "R" H 2950 4400 79  0000 C CNN
+F 1 "24k" H 2950 4400 79  0000 C CNN
 F 2 "" H 2850 4425 60  0001 C CNN
 F 3 "" H 2975 4225 60  0001 C CNN
@@
 P 2950 5000
 F 0 "R12" H 2950 5150 79  0000 C CNN
-F 1 "R" H 2950 5000 79  0000 C CNN
+F 1 "56.2k" H 2950 5000 79  0000 C CNN
 F 2 "" H 2850 5025 60  0001 C CNN
 F 3 "" H 2975 4825 60  0001 C CNN
@@
 P 2950 5600
 F 0 "R13" H 2950 5750 79  0000 C CNN
-F 1 "R" H 2950 5600 79  0000 C CNN
+F 1 "33.2k" H 2950 5600 79  0000 C CNN
 F 2 "" H 2850 5625 60  0001 C CNN
 F 3 "" H 2975 5425 60  0001 C CNN
@@
 P 2200 6250
 F 0 "R8" H 2200 6400 79  0000 C CNN
-F 1 "R" H 2200 6250 79  0000 C CNN
+F 1 "12k" H 2200 6250 79  0000 C CNN
 F 2 "" H 2100 6275 60  0001 C CNN
 F 3 "" H 2225 6075 60  0001 C CNN
@@
 Connection ~ 4750 2200
 Wire Wire Line
-	1650 6250 1850 6250
+	1650 6250 1775 6250
 Wire Wire Line
 	3300 4400 3600 4400
@@
 Wire Wire Line
 	3600 5000 3600 5600
-$Comp
-L Amplifier_Operational_GOST:140УД20 D2
-U 1 1 67D27BAE
-P 5000 4800
-F 0 "D2" H 5000 5495 79  0000 C CNN
-F 1 "140УД20" H 5000 4100 79  0001 C CNN
-F 2 "Package_CDFP_RU:401.14-5" H 5050 3950 79  0001 C CNN
-F 3 "http://www.voshod-krlz.ru/files/datasheets/140UD20.pdf" H 6000 4850 79  0001 C CNN
-	1    5000 4800
-	1    0    0    -1
-$EndComp
 $Comp
 L Device_GOST:R R15
@@
 P 7300 2850
 F 0 "R15" V 7050 3050 79  0000 C CNN
-F 1 "R" H 7300 2850 79  0000 C CNN
+F 1 "2.05k" H 7300 2850 79  0000 C CNN
 F 2 "" H 7200 2875 60  0001 C CNN
 F 3 "" H 7325 2675 60  0001 C CNN
@@
 P 7300 3700
 F 0 "R14" V 7050 3900 79  0000 C CNN
-F 1 "R" H 7300 3700 79  0000 C CNN
+F 1 "10k" H 7300 3700 79  0000 C CNN
 F 2 "" H 7200 3725 60  0001 C CNN
 F 3 "" H 7325 3525 60  0001 C CNN
@@
 P 7950 3700
 F 0 "C3" H 8000 3800 79  0000 L CNN
-F 1 "C" H 8050 3600 79  0000 L CNN
+F 1 "15" H 8050 3600 79  0000 L CNN
 F 2 "" H 7875 3700 60  0001 C CNN
 F 3 "" H 7975 3800 60  0001 C CNN
@@
 P 7850 2400
 F 0 "R98" H 7950 2600 79  0000 C CNN
-F 1 "R" H 7850 2400 79  0000 C CNN
+F 1 "2M" H 7850 2400 79  0000 C CNN
 F 2 "" H 7750 2425 60  0001 C CNN
 F 3 "" H 7875 2225 60  0001 C CNN
@@
 P 8650 2400
 F 0 "R28" H 8750 2600 79  0000 C CNN
-F 1 "R" H 8650 2400 79  0000 C CNN
+F 1 "8.2M" H 8650 2400 79  0000 C CNN
 F 2 "" H 8550 2425 60  0001 C CNN
 F 3 "" H 8675 2225 60  0001 C CNN
@@
 P 9450 2400
 F 0 "R29" H 9550 2600 79  0000 C CNN
-F 1 "R" H 9450 2400 79  0000 C CNN
+F 1 "10M" H 9450 2400 79  0000 C CNN
 F 2 "" H 9350 2425 60  0001 C CNN
 F 3 "" H 9475 2225 60  0001 C CNN
@@
 Wire Wire Line
 	9000 2400 9100 2400
-$Comp
-L Amplifier_Operational_GOST:140УД20 D4
-U 1 1 67CE1C12
-P 10800 2800
-F 0 "D4" H 10800 3495 79  0000 C CNN
-F 1 "140УД20" H 10800 2100 79  0001 C CNN
-F 2 "Package_CDFP_RU:401.14-5" H 10850 1950 79  0001 C CNN
-F 3 "http://www.voshod-krlz.ru/files/datasheets/140UD20.pdf" H 11800 2850 79  0001 C CNN
-	1    10800 2800
-	1    0    0    -1
-$EndComp
 Wire Wire Line
 	10350 1600 10000 1600
@@
 P 7700 4850
 F 0 "C9" H 7750 4950 79  0000 L CNN
-F 1 "C" H 7800 4750 79  0000 L CNN
+F 1 "6.8" H 7800 4750 79  0000 L CNN
 F 2 "" H 7625 4850 60  0001 C CNN
 F 3 "" H 7725 4950 60  0001 C CNN
@@
 P 10100 5250
 F 0 "VD10" H 9800 5050 79  0000 L CNN
-F 1 "VD" H 10100 5050 79  0001 C CNN
+F 1 "2Д522Б" H 10100 5050 79  0001 C CNN
 F 2 "" H 10002 5250 79  0001 C CNN
 F 3 "" H 10002 5250 79  0001 C CNN
@@
 P 10100 4400
 F 0 "VD9" H 10250 4500 79  0000 L CNN
-F 1 "VD" H 10100 4200 79  0001 C CNN
+F 1 "2Д522Б" H 10100 4200 79  0001 C CNN
 F 2 "" H 10002 4400 79  0001 C CNN
 F 3 "" H 10002 4400 79  0001 C CNN
@@
 P 8700 4400
 F 0 "R43" H 8700 4550 79  0000 C CNN
-F 1 "R" H 8700 4400 79  0000 C CNN
+F 1 "2.91k" H 8700 4400 79  0000 C CNN
 F 2 "" H 8600 4425 60  0001 C CNN
 F 3 "" H 8725 4225 60  0001 C CNN
@@
 P 11200 4400
 F 0 "R54" H 11200 4550 79  0000 C CNN
-F 1 "R" H 11200 4400 79  0000 C CNN
+F 1 "130" H 11200 4400 79  0000 C CNN
 F 2 "" H 11100 4425 60  0001 C CNN
 F 3 "" H 11225 4225 60  0001 C CNN
@@
 P 11200 5250
 F 0 "R55" H 11200 5400 79  0000 C CNN
-F 1 "R" H 11200 5250 79  0000 C CNN
+F 1 "130" H 11200 5250 79  0000 C CNN
 F 2 "" H 11100 5275 60  0001 C CNN
 F 3 "" H 11225 5075 60  0001 C CNN
@@
 P 10150 6000
 F 0 "R50" H 10150 6150 79  0000 C CNN
-F 1 "R" H 10150 6000 79  0000 C CNN
+F 1 "3.92k" H 10150 6000 79  0000 C CNN
 F 2 "" H 10050 6025 60  0001 C CNN
 F 3 "" H 10175 5825 60  0001 C CNN
@@
 L power_GOST:+12V #PWR?
 U 1 1 67D0D101
-P 6550 3350
-F 0 "#PWR?" H 6550 3250 79  0001 C CNN
-F 1 "+12V" H 6400 3600 79  0000 L CNN
-F 2 "" V 6550 3475 98  0000 C CNN
-F 3 "" H 6550 3475 98  0001 C CNN
-	1    6550 3350
-	-1   0    0    1
+P 6100 3000
+F 0 "#PWR?" H 6100 2900 79  0001 C CNN
+F 1 "+12V" V 6050 3100 79  0000 L CNN
+F 2 "" V 6100 3125 98  0000 C CNN
+F 3 "" H 6100 3125 98  0001 C CNN
+	1    6100 3000
+	0    1    1    0
 $EndComp
 $Comp
@@
 P 6500 2600
 F 0 "R20" H 6900 2700 79  0000 C CNN
-F 1 "R" H 6500 2600 79  0000 C CNN
+F 1 "5.05k" H 6500 2600 79  0000 C CNN
 F 2 "" H 6400 2625 60  0001 C CNN
 F 3 "" H 6525 2425 60  0001 C CNN
@@
 P 6500 2800
 F 0 "R22" H 6900 2900 79  0000 C CNN
-F 1 "R" H 6500 2800 79  0000 C CNN
+F 1 "5.05k" H 6500 2800 79  0000 C CNN
 F 2 "" H 6400 2825 60  0001 C CNN
 F 3 "" H 6525 2625 60  0001 C CNN
@@
 P 6700 4400
 F 0 "R36" H 6700 4550 79  0000 C CNN
-F 1 "R" H 6700 4400 79  0000 C CNN
+F 1 "1.01k" H 6700 4400 79  0000 C CNN
 F 2 "" H 6600 4425 60  0001 C CNN
 F 3 "" H 6725 4225 60  0001 C CNN
@@
 F1 "upr.sch" 50
 $EndSheet
-Wire Wire Line
-	6550 3000 6550 3350
-Wire Wire Line
-	6100 3000 6550 3000
-Wire Wire Line
-	6550 3000 7050 3000
-Wire Wire Line
-	7050 3000 7050 2800
-Connection ~ 6550 3000
 Connection ~ 7050 2800
 $Sheet
@@
 P 2100 5600
 F 0 "R6" H 2100 5750 79  0000 C CNN
-F 1 "R" H 2100 5600 79  0000 C CNN
+F 1 "180k" H 2100 5600 79  0000 C CNN
 F 2 "" H 2000 5625 60  0001 C CNN
 F 3 "" H 2125 5425 60  0001 C CNN
@@
 Text Notes 8050 2200 0    50   ~ 0
 *
+Wire Wire Line
+	7050 3200 6200 3200
+Wire Wire Line
+	7050 2800 7050 3200
+Connection ~ 6200 3200
+$Comp
+L Amplifier_Operational_GOST:140УД6А DA1
+U 1 1 67CEE261
+P 5500 2800
+F 0 "DA1" H 5500 3495 79  0000 C CNN
+F 1 "140УД6А" H 5500 2100 50  0001 C CNN
+F 2 "Package_TO_SOT_THT_RU:3101.8" H 5500 2000 50  0001 C CNN
+F 3 "" H 5500 2800 50  0001 C CNN
+	1    5500 2800
+	1    0    0    -1
+$EndComp
+$Comp
+L Amplifier_Operational_GOST:140УД6А DA2
+U 1 1 67CF11E3
+P 5000 4800
+F 0 "DA2" H 5000 5495 79  0000 C CNN
+F 1 "140УД6А" H 5000 4100 50  0001 C CNN
+F 2 "Package_TO_SOT_THT_RU:3101.8" H 5000 4000 50  0001 C CNN
+F 3 "" H 5000 4800 50  0001 C CNN
+	1    5000 4800
+	1    0    0    -1
+$EndComp
+$Comp
+L Amplifier_Operational_GOST:140УД6А DA4
+U 1 1 67CF187F
+P 10800 2800
+F 0 "DA4" H 10800 3495 79  0000 C CNN
+F 1 "544УД1А" H 10800 2100 50  0001 C CNN
+F 2 "Package_TO_SOT_THT_RU:3101.8" H 10800 2000 50  0001 C CNN
+F 3 "" H 10800 2800 50  0001 C CNN
+	1    10800 2800
+	1    0    0    -1
+$EndComp
+$Comp
+L power_GOST:GND #PWR?
+U 1 1 67D5B8F1
+P 1775 6375
+F 0 "#PWR?" H 1775 6425 60  0001 C CNN
+F 1 "GND" H 1775 6125 79  0001 C CNN
+F 2 "" H 1775 6375 60  0000 C CNN
+F 3 "" H 1775 6375 60  0001 C CNN
+	1    1775 6375
+	1    0    0    -1
+$EndComp
+Wire Wire Line
+	1775 6250 1775 6375
+Connection ~ 1775 6250
+Wire Wire Line
+	1775 6250 1850 6250
 $EndSCHEMATC
