File: EP-528_ser.2/EP-528_ser.2/Pit.sch (KiCad schematic (older format))
At the start: 90 parts, among them X13 CON, X17 CON, X18 CON, X19 CON, X2 CON, X25 CON, X26 CON, X3 CON, X35 CON, X4 CON, X45 CON, X48 CON, X49 CON, X6 CON, X7 CON

Commit message: Обновлены файлы ЭП
Parts:
- removed VD? (x24): VD, symbol Device_GOST:VD
- added VD11, VD12, VD17, VD18, VD19, VD20: 2Д906А_свыводами, Diode_THT_RU:2Д906А, symbol Diode_GOST:2Д906А_свыводами
- C10: value C -> 0.022
- C11, C20: value CP -> 15
- C14, C15, C16, C17, C18, C19, C4: value CP -> 33
- R1: value R -> 27
- R10, R48: value R -> 3.9k
- R24: value R -> 300
- R26: value R -> 470
- R27: value R -> 1.2k
- R40: value R -> 5.1k
- R44, R45: value R -> 2.2k
- R51: value R -> 240
- R52: value R -> 294
- R53: value R -> 4.02
- R58: value R -> 180
- R71, R76: value R -> 20
- R79, R82: value R -> 33
- R85, R87: value R -> 43
- R86: value R -> 510
- R88: value R -> 75
- R89: value R -> 3k
- R90: value R -> 1.8k
- R91: value R -> 910
- VD8: value VD_ZENER -> Д818Г
- VT1: value VT_NPN_BCE -> 2Т827А
- VT10: renamed from VT2; value VT_NPN_BCE -> 2Т630Б
- VT2, VT3: value VT_NPN_BCE -> 2Т630Б
Connections:
- wire segments 210 -> 239
Other:
- note added: "22"
- note removed: "27"
