File: EP-528_ser.2/EP-528_ser.2/upr.sch (KiCad schematic (older format))
At the start: 103 parts, among them X11 CON, X12 CON, X20 CON, X21 CON, X24 CON, X27 CON, X28 CON, X29 CON, X30 CON, X31 CON, X33 CON, X33.1 CON, X34 CON, X36 CON, X37 CON, X38 CON, X39 CON, X39.1 CON, X40 CON, X41 CON, X42 CON, X43 CON, X50 CON, X8 CON

Commit message: Обновлены файлы ЭП
Parts:
- removed D3, D5, D6: 140УД20, Package_CDFP_RU:401.14-5, symbol Amplifier_Operational_GOST:140УД20
- removed VD? (x8): VD, symbol Device_GOST:VD
- added DA3, DA5, DA6: 140УД6А, Package_TO_SOT_THT_RU:3101.8, symbol Amplifier_Operational_GOST:140УД6А
- added VD15, VD16: 2Д906А_свыводами, Diode_THT_RU:2Д906А, symbol Diode_GOST:2Д906А_свыводами
- C1: value C -> 47
- C12: value C -> 150
- C13: value CP -> 150
- C5: value C -> 0.068
- C6, C7: value C -> 6.8
- R16, R4: value R -> 10k
- R17: value R -> 750k
- R18: value R -> 36k
- R19: value R -> 3k
- R21, R23: value R -> 5.05k
- R3: value R -> 316k
- R30, R31, R32, R33: value R -> 5.11k
- R34, R35: value R -> 2k
- R38, R39: value R -> 8.16k
- R41, R42: value R -> 115k
- R46, R47: value R -> 2M
- R5: value R -> 110
- R56, R57: value R -> 5.6k
- R59, R60: value R -> 390k
- R61, R62: value R -> 330k
- R63, R64, R65, R66: value R -> 2.7k
- R67, R68: value R -> 17.4k
- R69, R70: value R -> 1k
- R72, R73: value R -> 68k
- R74, R75: value R -> 22.6k
- R77, R78: value R -> 54.9k
- R80, R81: value R -> 130k
- R83, R84: value R -> 243k
- R92, R93: value R -> 11k
- R94, R95: value R -> 1.3M
- R96, R97: value R -> 2m?
- VD13, VD14: value VD -> 2Д213А
- VD2, VD21, VD3: value VD -> 2Д522Б
- VT4, VT5: value VT_NPN_BCE -> 2Т630Б
- VT6, VT7: value VT_PNP_BCE -> 2Т203Г
- VT8, VT9: value VT_PNP_BCE -> 2Т825А
Connections:
- wire segments 277 -> 283
